Commit message: Add collision and inertial properties

File: src/ddr_description/urdf/ddr_robot.urdf.xacro (robot description, xacro)
@@ -11,4 +11,14 @@
             <material name="blue" />
         </visual>
+        <collision>
+            <geometry>
+                <box size="${base_length} ${base_width} ${base_height}" />
+            </geometry>
+            <origin xyz="0 0 ${base_height / 2.0}" rpy="0 0 0" />
+        </collision>
+        <xacro:inertial_box mass="${base_mass}" x="${base_length}" y="${base_width}"
+                                z="${base_height}">
+                            <origin xyz="0 0 ${base_height / 2.0}" rpy="0 0 0" />
+        </xacro:inertial_box>
     </link>
     <xacro:macro name="wheel_link" params="prefix">
@@ -21,4 +31,14 @@
                 <material name="grey" />
             </visual>
+            <collision>
+                <geometry>
+                    <cylinder radius="${wheel_radius}" length="${wheel_length}" />
+                </geometry>
+                <origin xyz="0 0 0" rpy="${pi / 2.0} 0 0" />
+            </collision>
+            <xacro:inertial_cylinder mass="${wheel_mass}" length="${wheel_length}"
+                                                        radius="${wheel_radius}">
+                                    <origin xyz="0 0 0" rpy="${pi / 2.0} 0 0" />
+            </xacro:inertial_cylinder>
         </link>
     </xacro:macro>
@@ -33,4 +53,14 @@
             <material name="red" />
         </visual>
+        <collision>
+            <geometry>
+                <sphere radius="${caster_radius}" />
+            </geometry>
+            <origin xyz="0 0 0" rpy="0 0 0" />
+        </collision>
+        <xacro:inertial_sphere mass="${caster_mass}"
+                               radius="${caster_radius}">
+                               <origin xyz="0 0 0" rpy="0 0 0"/>
+        </xacro:inertial_sphere>
     </link>
     <link name="laser_link">
@@ -42,4 +72,14 @@
             <material name="dark_grey" />
         </visual>
+        <collision>
+            <geometry>
+                <cylinder radius="${lidar_radius}" length="${lidar_length}" />
+            </geometry>
+            <origin xyz="0 0 0" rpy="0 0 0" />
+        </collision>
+        <xacro:inertial_cylinder mass="${lidar_mass}" length="${lidar_length}"
+                                                      radius="${lidar_radius}">
+                                <origin xyz="0 0 0" rpy="0 0 0" />
+        </xacro:inertial_cylinder>
     </link>
     <link name="camera_link">
@@ -51,4 +91,14 @@
             <material name="green" />
         </visual>
+        <collision>
+             <geometry>
+                <box size="${camera_length} ${camera_width} ${camera_height}" />
+            </geometry>
+            <origin xyz="0 0 0" rpy="0 ${pi / 2.0} 0" />
+        </collision>
+        <xacro:inertial_box mass="${camera_mass}" x="${camera_length}" y="${camera_width}"
+                                z="${camera_height}">
+                            <origin xyz="0 0 0" rpy="0 ${pi / 2.0} 0" />
+        </xacro:inertial_box>
     </link>
     <link name="imu_link">
@@ -60,4 +110,14 @@
             <material name="blue" />
         </visual>
+        <collision>
+            <geometry>
+                <box size="${imu_length} ${imu_width} ${imu_height}" />
+            </geometry>
+            <origin xyz="0 0 0" rpy="0 0 0" />
+        </collision>
+        <xacro:inertial_box mass="${imu_mass}" x="${imu_length}" y="${imu_width}"
+                                z="${imu_height}">
+                            <origin xyz="0 0 0" rpy="0 0 0" />
+        </xacro:inertial_box>
     </link>
     <joint name="base_joint" type="fixed">

File: src/ddr_description/urdf/properties.xacro (robot description, xacro)
@@ -5,19 +5,25 @@
     <xacro:property name="base_width" value="0.4" />
     <xacro:property name="base_height" value="0.2" />
+    <xacro:property name="base_mass" value="8.0" />
     <!-- Wheels -->
     <xacro:property name="wheel_radius" value="0.1" />
     <xacro:property name="wheel_length" value="0.05" />
+    <xacro:property name="wheel_mass" value="0.5" />
     <xacro:property name="caster_radius" value="${wheel_radius / 2.0}" />
+    <xacro:property name="caster_mass" value="0.2" />
     <!-- LiDAR -->
     <xacro:property name="lidar_radius" value="0.0484" />
     <xacro:property name="lidar_length" value="0.0403" />
+    <xacro:property name="lidar_mass" value="0.1" />
     <!-- Camera -->
     <xacro:property name="camera_length" value="0.025" />
     <xacro:property name="camera_width" value="0.024" />
     <xacro:property name="camera_height" value="0.009" />
+    <xacro:property name="camera_mass" value="0.05" />
     <!-- IMU -->
     <xacro:property name="imu_length" value="0.04" />
     <xacro:property name="imu_width" value="0.03" />
     <xacro:property name="imu_height" value="0.01" />
+    <xacro:property name="imu_mass" value="0.02" />
     <!-- Materials -->
     <material name="red">
@@ -36,3 +42,30 @@
         <color rgba="0.3 0.3 0.3 1" />
     </material>
+    <xacro:macro name="inertial_box" params="mass x y z *origin">
+        <inertial>
+            <xacro:insert_block name="origin"/>
+            <mass value="${mass}" />
+            <inertia ixx="${(1/12) * mass * (y*y+z*z)}" ixy="0.0" ixz="0.0"
+                    iyy="${(1/12) * mass * (x*x+z*z)}" iyz="0.0"
+                    izz="${(1/12) * mass * (x*x+y*y)}" />
+        </inertial>
+    </xacro:macro>
+    <xacro:macro name="inertial_cylinder" params="mass length radius *origin">
+        <inertial>
+            <xacro:insert_block name="origin"/>
+            <mass value="${mass}" />
+            <inertia ixx="${(1/12) * mass * (3*radius*radius + length*length)}" ixy="0.0" ixz="0.0"
+                    iyy="${(1/12) * mass * (3*radius*radius + length*length)}" iyz="0.0"
+                    izz="${(1/2) * mass * (radius*radius)}" />
+        </inertial>
+    </xacro:macro>
+    <xacro:macro name="inertial_sphere" params="mass radius *origin">
+        <inertial>
+            <xacro:insert_block name="origin"/>
+            <mass value="${mass}" />
+            <inertia ixx="${(2/5) * mass * (radius*radius)}" ixy="0.0" ixz="0.0"
+                    iyy="${(2/5) * mass * (radius*radius)}" iyz="0.0"
+                    izz="${(2/5) * mass * (radius*radius)}" />
+        </inertial>
+    </xacro:macro>
 </robot>

Commit message: Add DDR diff drive controller

File: src/ddr_description/urdf/ddr_robot.urdf.xacro (robot description, xacro)
@@ -132,5 +132,5 @@
             <parent link="base_link" />
             <child link="${prefix}_wheel_link" />
-            <origin xyz="-0.15 ${sign * ((base_width / 2.0) + (wheel_length / 2.0))} 0" rpy="0 0 0" />
+            <origin xyz="-0.15 ${sign * wheel_separation / 2.0} 0" rpy="0 0 0" />
             <axis xyz="0 1 0" />
         </joint>

File: src/ddr_description/urdf/properties.xacro (robot description, xacro)
@@ -10,4 +10,5 @@
     <xacro:property name="wheel_length" value="0.05" />
     <xacro:property name="wheel_mass" value="0.5" />
+    <xacro:property name="wheel_separation" value="${base_width + wheel_length}" />
     <xacro:property name="caster_radius" value="${wheel_radius / 2.0}" />
     <xacro:property name="caster_mass" value="0.2" />

Commit message: Tune DDR simulation parameters

File: src/ddr_description/urdf/ddr_robot.urdf.xacro (robot description, xacro)
@@ -132,5 +132,5 @@
             <parent link="base_link" />
             <child link="${prefix}_wheel_link" />
-            <origin xyz="-0.15 ${sign * wheel_separation / 2.0} 0" rpy="0 0 0" />
+            <origin xyz="-${base_length / 4.0} ${sign * wheel_separation / 2.0} 0" rpy="0 0 0" />
             <axis xyz="0 1 0" />
         </joint>
@@ -141,5 +141,5 @@
         <parent link="base_link" />
         <child link="caster_wheel_link" />
-        <origin xyz="0.2 0 -${caster_radius}" rpy="0 0 0" />
+        <origin xyz="${base_length / 3.0} 0 -${caster_radius}" rpy="0 0 0" />
     </joint>
     <joint name="laser_joint" type="fixed">

File: src/ddr_description/urdf/gazebo.xacro (robot description, xacro)
@@ -3,6 +3,6 @@
     <!-- Wheels -->
     <gazebo reference="right_wheel_link">
-        <mu1>1000000000000000.0</mu1>
-        <mu2>1000000000000000.0</mu2>
+        <mu1>5.0</mu1>
+        <mu2>5.0</mu2>
         <kp>1000000000000.0</kp>
         <kd>10.0</kd>
@@ -12,6 +12,6 @@
     </gazebo>
     <gazebo reference="left_wheel_link">
-        <mu1>1000000000000000.0</mu1>
-        <mu2>1000000000000000.0</mu2>
+        <mu1>5.0</mu1>
+        <mu2>5.0</mu2>
         <kp>1000000000000.0</kp>
         <kd>10.0</kd>
@@ -22,6 +22,6 @@
     <!-- Caster Wheels -->
     <gazebo reference="caster_wheel_link">
-        <mu1>0.1</mu1>
-        <mu2>0.1</mu2>
+        <mu1>0.3</mu1>
+        <mu2>0.3</mu2>
         <kp>1000000.0</kp>
         <kd>100.0</kd>

File: src/ddr_description/urdf/ros2_control.xacro (robot description, xacro)
@@ -9,6 +9,6 @@
         <joint name="right_wheel_joint">
             <command_interface name="velocity">
-              <param name="min">-1</param>
-              <param name="max">1</param>
+              <param name="min">-5</param>
+              <param name="max">5</param>
             </command_interface>
             <state_interface name="position" />
@@ -17,6 +17,6 @@
         <joint name="left_wheel_joint">
             <command_interface name="velocity">
-              <param name="min">-1</param>
-              <param name="max">1</param>
+              <param name="min">-5</param>
+              <param name="max">5</param>
             </command_interface>
             <state_interface name="position" />

Commit message: Add camera optical frame

File: src/ddr_description/urdf/ddr_robot.urdf.xacro (robot description, xacro)
@@ -85,4 +85,5 @@
         </xacro:inertial_cylinder>
     </link>
+    <link name="camera_optical_frame" />
     <link name="camera_link">
         <visual>
@@ -148,4 +149,9 @@
         <origin xyz="0 0 ${base_height + lidar_length / 2.0}" rpy="0 0 0" />
     </joint>
+    <joint name="camera_optical_joint" type="fixed">
+        <parent link="camera_link" />
+        <child link="camera_optical_frame" />
+        <origin xyz="0 0 0" rpy="${-pi / 2.0} 0 ${-pi / 2.0}" />
+    </joint>
     <joint name="camera_joint" type="fixed">
         <parent link="base_link" />

File: src/ddr_description/urdf/gazebo.xacro (robot description, xacro)
@@ -70,5 +70,4 @@
         </sensor>
     </gazebo>
-    <!-- Camera -->
     <gazebo reference="camera_link">
         <sensor name="camera_sensor" type="camera">
@@ -77,4 +76,5 @@
             <visualize>true</visualize>
             <topic>camera/image</topic>
+            <gz_frame_id>camera_optical_frame</gz_frame_id>
             <camera>
                 <horizontal_fov>1.047</horizontal_fov>
